Commit message: Updated diffbot_description sizes

File: description/urdf/diffbot_description.urdf.xacro (robot description, xacro)
@@ -4,11 +4,11 @@
   <!-- Constants for robot dimensions -->
   <xacro:property name="PI" value="3.1415926535897931"/>
-  <xacro:property name="base_mass" value="0.3" /> <!-- arbitrary value for base mass -->
-  <xacro:property name="base_width" value="0.1" />
-  <xacro:property name="base_length" value="0.1" />
-  <xacro:property name="base_height" value="0.05" />
-  <xacro:property name="wheel_mass" value="0.3" /> <!-- arbitrary value for wheel mass -->
-  <xacro:property name="wheel_len" value="0.020" />
-  <xacro:property name="wheel_radius" value="0.015" />
+  <xacro:property name="base_mass" value="1.0" /> <!-- arbitrary value for base mass -->
+  <xacro:property name="base_width" value="0.12" />
+  <xacro:property name="base_length" value="0.2" />
+  <xacro:property name="base_height" value="0.1" />
+  <xacro:property name="wheel_mass" value="0.7" /> <!-- arbitrary value for wheel mass -->
+  <xacro:property name="wheel_len" value="0.040" />
+  <xacro:property name="wheel_radius" value="0.05" />
   <xacro:property name="caster_wheel_mass" value="0.1" /> <!-- arbitrary value for caster wheel mass -->
   <xacro:property name="caster_wheel_radius" value="0.015" />

Commit message: Updated left wheel origin orientation

File: description/urdf/diffbot_description.urdf.xacro (robot description, xacro)
@@ -41,5 +41,5 @@
       <parent link="${prefix}base_link"/>
       <child link="${prefix}left_wheel"/>
-      <origin xyz="0 -${base_width/2} ${z_offset}" rpy="0 0 0"/>
+      <origin xyz="0 -${base_width/2} ${z_offset}" rpy="-${pi/2} 0 0"/>
       <axis xyz="0 1 0"/>
       <dynamics damping="0.2"/>

Commit message: updated left wheel axis rotation

File: description/urdf/diffbot_description.urdf.xacro (robot description, xacro)
@@ -41,6 +41,6 @@
       <parent link="${prefix}base_link"/>
       <child link="${prefix}left_wheel"/>
-      <origin xyz="0 -${base_width/2} ${z_offset}" rpy="-${pi/2} 0 0"/>
-      <axis xyz="0 1 0"/>
+      <origin xyz="0 -${base_width/2} ${z_offset}" rpy="0 0 0"/>
+      <axis xyz="0 0 1"/>
       <dynamics damping="0.2"/>
     </joint>

Commit message: Updated robot urdf

File: description/urdf/diffbot_description.urdf.xacro (robot description, xacro)
@@ -6,5 +6,5 @@
   <xacro:property name="base_mass" value="1.0" /> <!-- arbitrary value for base mass -->
   <xacro:property name="base_width" value="0.12" />
-  <xacro:property name="base_length" value="0.2" />
+  <xacro:property name="base_length" value="0.25" />
   <xacro:property name="base_height" value="0.1" />
   <xacro:property name="wheel_mass" value="0.7" /> <!-- arbitrary value for wheel mass -->
@@ -19,5 +19,5 @@
       <origin xyz="0 0 0" rpy="0 0 0"/>
       <geometry>
-        <box size="${base_width} ${base_length} ${base_height}"/>
+        <box size="${base_length} ${base_width} ${base_height}"/>
       </geometry>
     </collision>
@@ -25,5 +25,5 @@
       <origin xyz="0 0 ${base_height/2}" rpy="0 0 0"/>
       <geometry>
-        <box size="${base_width} ${base_length} ${base_height}"/>
+        <box size="${base_length} ${base_width} ${base_height}"/>
       </geometry>
       <material name="orange"/>
@@ -41,6 +41,6 @@
       <parent link="${prefix}base_link"/>
       <child link="${prefix}left_wheel"/>
-      <origin xyz="0 -${base_width/2} ${z_offset}" rpy="0 0 0"/>
-      <axis xyz="0 0 1"/>
+      <origin xyz="${base_length/2-wheel_radius} -${base_width/2+wheel_len/2} 0" rpy="${PI} 0 0"/>
+      <axis xyz="0 1 0"/>
       <dynamics damping="0.2"/>
     </joint>
@@ -72,5 +72,5 @@
       <parent link="${prefix}base_link"/>
       <child link="${prefix}right_wheel"/>
-      <origin xyz="0 ${base_width/2} ${z_offset}" rpy="0 0 0"/>
+      <origin xyz="${base_length/2-wheel_radius} ${base_width/2+wheel_len/2} 0" rpy="0 0 0"/>
       <axis xyz="0 1 0"/>
       <dynamics damping="0.2"/>
@@ -98,33 +98,4 @@
           iyy="${wheel_mass / 12.0 * wheel_radius*wheel_radius}" iyz="0.0"
           izz="${wheel_mass / 12.0 * wheel_radius*wheel_radius}"/>
-        </inertial>
-      </link>
-    <joint name="${prefix}caster_frontal_wheel_joint" type="fixed">
-      <parent link="${prefix}base_link"/>
-      <child link="${prefix}caster_frontal_wheel"/>
-      <origin xyz="${base_width/2 - caster_wheel_radius} 0 ${z_offset}" rpy="0 0 0"/>
-    </joint>
-    <!-- caster frontal wheel Link -->
-    <link name="${prefix}caster_frontal_wheel">
-      <collision>
-        <origin xyz="0 0 0" rpy="0 0 0"/>
-        <geometry>
-          <sphere radius="${caster_wheel_radius}"/>
-        </geometry>
-      </collision>
-      <visual>
-        <origin xyz="0 0 0" rpy="0 0 0"/>
-        <geometry>
-          <sphere radius="${caster_wheel_radius}"/>
-        </geometry>
-        <material name="white"/>
-      </visual>
-      <inertial>
-        <origin xyz="0 0 0" rpy="0 0 0"/>
-        <mass value="${caster_wheel_mass}"/>
-        <inertia
-          ixx="${caster_wheel_mass * 0.4 * (caster_wheel_radius * caster_wheel_radius)}" ixy="0.0" ixz="0.0"
-          iyy="${caster_wheel_mass * 0.4 * (caster_wheel_radius * caster_wheel_radius)}" iyz="0.0"
-          izz="${caster_wheel_mass * 0.4 * (caster_wheel_radius * caster_wheel_radius)}"/>
         </inertial>
       </link>

File: description/urdf/lidar.xacro (robot description, xacro)
@@ -4,5 +4,5 @@
         <parent link="base_link"/>
         <child link="laser_frame"/>
-        <origin xyz="0.1 0 0.175" rpy="0 0 0"/>
+        <origin xyz="0.1 0 0.125" rpy="0 0 0"/>
     </joint>
     <link name="laser_frame">

Commit message: updated robot urdf

File: description/urdf/diffbot_description.urdf.xacro (robot description, xacro)
@@ -12,5 +12,5 @@
   <xacro:property name="wheel_radius" value="0.05" />
   <xacro:property name="caster_wheel_mass" value="0.1" /> <!-- arbitrary value for caster wheel mass -->
-  <xacro:property name="caster_wheel_radius" value="0.015" />
+  <xacro:property name="caster_wheel_radius" value="0.0015" />
   <xacro:property name="z_offset" value="-${base_height/2}" /> <!-- Space btw top of beam and the each joint -->
   <!-- Base Link -->

Commit message: setting up params for SLAM toolbox

File: description/urdf/diffbot_description.urdf.xacro (robot description, xacro)
@@ -36,5 +36,13 @@
         iyy="${base_mass / 12.0 * (base_height*base_height + base_width*base_width)}" iyz="0.0"
         izz="${base_mass / 12.0 * (base_width*base_width + base_length*base_length)}"/>
-      </inertial>
+    </inertial>
+  </link>
+  <!-- BASE_FOOTPRINT LINK -->
+  <joint name="base_footprint_joint" type="fixed">
+        <parent link="${prefix}base_link"/>
+        <child link="base_footprint"/>
+        <origin xyz="0 0 0" rpy="0 0 0"/>
+    </joint>
+    <link name="base_footprint">
     </link>
     <joint name="${prefix}left_wheel_joint" type="continuous">

Commit message: Updated lidar and robot xacro

File: description/urdf/diffbot_description.urdf.xacro (robot description, xacro)
@@ -49,5 +49,5 @@
       <parent link="${prefix}base_link"/>
       <child link="${prefix}left_wheel"/>
-      <origin xyz="${base_length/2-wheel_radius} -${base_width/2+wheel_len/2} 0" rpy="${PI} 0 0"/>
+      <origin xyz="-${base_length/2-wheel_radius} -${base_width/2+wheel_len/2} 0" rpy="0 0 0"/>
       <axis xyz="0 1 0"/>
       <dynamics damping="0.2"/>
@@ -80,5 +80,5 @@
       <parent link="${prefix}base_link"/>
       <child link="${prefix}right_wheel"/>
-      <origin xyz="${base_length/2-wheel_radius} ${base_width/2+wheel_len/2} 0" rpy="0 0 0"/>
+      <origin xyz="-${base_length/2-wheel_radius} ${base_width/2+wheel_len/2} 0" rpy="${PI} 0 0"/>
       <axis xyz="0 1 0"/>
       <dynamics damping="0.2"/>
@@ -111,5 +111,5 @@
       <parent link="${prefix}base_link"/>
       <child link="${prefix}caster_rear_wheel"/>
-      <origin xyz="${-base_width/2 + caster_wheel_radius} 0 ${z_offset}" rpy="0 0 0"/>
+      <origin xyz="-${-base_width/2 + caster_wheel_radius} 0 ${z_offset}" rpy="0 0 0"/>
     </joint>
     <!-- caster rear wheel Link -->

File: description/urdf/lidar.xacro (robot description, xacro)
@@ -9,5 +9,5 @@
         <visual>
             <geometry>
-                <cylinder radius="0.05" length="0.04"/>
+                <cylinder radius="0.03" length="0.04"/>
             </geometry>
             <material name="red"/>

Commit message: Updated robot urdf

File: description/urdf/diffbot_description.urdf.xacro (robot description, xacro)
@@ -4,13 +4,13 @@
   <!-- Constants for robot dimensions -->
   <xacro:property name="PI" value="3.1415926535897931"/>
-  <xacro:property name="base_mass" value="1.0" /> <!-- arbitrary value for base mass -->
-  <xacro:property name="base_width" value="0.12" />
-  <xacro:property name="base_length" value="0.25" />
-  <xacro:property name="base_height" value="0.1" />
-  <xacro:property name="wheel_mass" value="0.7" /> <!-- arbitrary value for wheel mass -->
+  <xacro:property name="base_mass" value="0.3" /> <!-- arbitrary value for base mass -->
+  <xacro:property name="base_width" value="0.1" />
+  <xacro:property name="base_length" value="0.1" />
+  <xacro:property name="base_height" value="0.05" />
+  <xacro:property name="wheel_mass" value="0.3" /> <!-- arbitrary value for wheel mass -->
   <xacro:property name="wheel_len" value="0.040" />
   <xacro:property name="wheel_radius" value="0.05" />
   <xacro:property name="caster_wheel_mass" value="0.1" /> <!-- arbitrary value for caster wheel mass -->
-  <xacro:property name="caster_wheel_radius" value="0.0015" />
+  <xacro:property name="caster_wheel_radius" value="0.005" />
   <xacro:property name="z_offset" value="-${base_height/2}" /> <!-- Space btw top of beam and the each joint -->
   <!-- Base Link -->
@@ -19,5 +19,5 @@
       <origin xyz="0 0 0" rpy="0 0 0"/>
       <geometry>
-        <box size="${base_length} ${base_width} ${base_height}"/>
+        <box size="${base_width} ${base_length} ${base_height}"/>
       </geometry>
     </collision>
@@ -25,5 +25,5 @@
       <origin xyz="0 0 ${base_height/2}" rpy="0 0 0"/>
       <geometry>
-        <box size="${base_length} ${base_width} ${base_height}"/>
+        <box size="${base_width} ${base_length} ${base_height}"/>
       </geometry>
       <material name="orange"/>
@@ -36,18 +36,10 @@
         iyy="${base_mass / 12.0 * (base_height*base_height + base_width*base_width)}" iyz="0.0"
         izz="${base_mass / 12.0 * (base_width*base_width + base_length*base_length)}"/>
-    </inertial>
-  </link>
-  <!-- BASE_FOOTPRINT LINK -->
-  <joint name="base_footprint_joint" type="fixed">
-        <parent link="${prefix}base_link"/>
-        <child link="base_footprint"/>
-        <origin xyz="0 0 0" rpy="0 0 0"/>
-    </joint>
-    <link name="base_footprint">
+      </inertial>
     </link>
     <joint name="${prefix}left_wheel_joint" type="continuous">
       <parent link="${prefix}base_link"/>
       <child link="${prefix}left_wheel"/>
-      <origin xyz="-${base_length/2-wheel_radius} -${base_width/2+wheel_len/2} 0" rpy="0 0 0"/>
+      <origin xyz="0 -${base_width/2} ${z_offset}" rpy="0 0 0"/>
       <axis xyz="0 1 0"/>
       <dynamics damping="0.2"/>
@@ -80,5 +72,5 @@
       <parent link="${prefix}base_link"/>
       <child link="${prefix}right_wheel"/>
-      <origin xyz="-${base_length/2-wheel_radius} ${base_width/2+wheel_len/2} 0" rpy="${PI} 0 0"/>
+      <origin xyz="0 ${base_width/2} ${z_offset}" rpy="0 0 0"/>
       <axis xyz="0 1 0"/>
       <dynamics damping="0.2"/>
@@ -108,8 +100,37 @@
         </inertial>
       </link>
+    <joint name="${prefix}caster_frontal_wheel_joint" type="fixed">
+      <parent link="${prefix}base_link"/>
+      <child link="${prefix}caster_frontal_wheel"/>
+      <origin xyz="${base_width/2 - caster_wheel_radius} 0 ${z_offset}" rpy="0 0 0"/>
+    </joint>
+    <!-- caster frontal wheel Link -->
+    <link name="${prefix}caster_frontal_wheel">
+      <collision>
+        <origin xyz="0 0 0" rpy="0 0 0"/>
+        <geometry>
+          <sphere radius="${caster_wheel_radius}"/>
+        </geometry>
+      </collision>
+      <visual>
+        <origin xyz="0 0 0" rpy="0 0 0"/>
+        <geometry>
+          <sphere radius="${caster_wheel_radius}"/>
+        </geometry>
+        <material name="white"/>
+      </visual>
+      <inertial>
+        <origin xyz="0 0 0" rpy="0 0 0"/>
+        <mass value="${caster_wheel_mass}"/>
+        <inertia
+          ixx="${caster_wheel_mass * 0.4 * (caster_wheel_radius * caster_wheel_radius)}" ixy="0.0" ixz="0.0"
+          iyy="${caster_wheel_mass * 0.4 * (caster_wheel_radius * caster_wheel_radius)}" iyz="0.0"
+          izz="${caster_wheel_mass * 0.4 * (caster_wheel_radius * caster_wheel_radius)}"/>
+        </inertial>
+      </link>
     <joint name="${prefix}caster_rear_wheel_joint" type="fixed">
       <parent link="${prefix}base_link"/>
       <child link="${prefix}caster_rear_wheel"/>
-      <origin xyz="-${-base_width/2 + caster_wheel_radius} 0 ${z_offset}" rpy="0 0 0"/>
+      <origin xyz="${-base_width/2 + caster_wheel_radius} 0 ${z_offset}" rpy="0 0 0"/>
     </joint>
     <!-- caster rear wheel Link -->

Commit message: Added Base_FootPRINT link

File: description/urdf/diffbot_description.urdf.xacro (robot description, xacro)
@@ -37,4 +37,12 @@
         izz="${base_mass / 12.0 * (base_width*base_width + base_length*base_length)}"/>
       </inertial>
+    </link>
+    <!-- BASE_FOOTPRINT LINK -->
+    <joint name="base_footprint_joint" type="fixed">
+        <parent link="${prefix}base_link"/>
+        <child link="base_footprint"/>
+        <origin xyz="0 0 0" rpy="0 0 0"/>
+    </joint>
+    <link name="base_footprint">
     </link>
     <joint name="${prefix}left_wheel_joint" type="continuous">

Commit message: Updated URDF

File: description/urdf/diffbot_description.urdf.xacro (robot description, xacro)
@@ -5,6 +5,6 @@
   <xacro:property name="PI" value="3.1415926535897931"/>
   <xacro:property name="base_mass" value="0.3" /> <!-- arbitrary value for base mass -->
-  <xacro:property name="base_width" value="0.1" />
-  <xacro:property name="base_length" value="0.1" />
+  <xacro:property name="base_width" value="0.15" />
+  <xacro:property name="base_length" value="0.3" />
   <xacro:property name="base_height" value="0.05" />
   <xacro:property name="wheel_mass" value="0.3" /> <!-- arbitrary value for wheel mass -->
@@ -49,5 +49,5 @@
       <parent link="${prefix}base_link"/>
       <child link="${prefix}left_wheel"/>
-      <origin xyz="0 ${base_width/2} 0" rpy="-${PI/2} 0 0"/>
+      <origin xyz="${base_length/2} ${base_width/2} 0" rpy="${PI/2} 0 0"/>
       <axis xyz="0 0 1"/>
       <dynamics damping="0.0"/>
@@ -78,5 +78,5 @@
       <parent link="${prefix}base_link"/>
       <child link="${prefix}right_wheel"/>
-      <origin xyz="0 ${-base_width/2} 0" rpy="${PI/2} 0 0"/>
+      <origin xyz="${base_length/2} ${-base_width/2} 0" rpy="${PI/2} 0 0"/>
       <axis xyz="0 0 -1"/>
       <dynamics damping="0.0"/>

Commit message: Updated URDF

File: description/urdf/diffbot_description.urdf.xacro (robot description, xacro)
@@ -7,5 +7,5 @@
   <xacro:property name="base_width" value="0.15" />
   <xacro:property name="base_length" value="0.3" />
-  <xacro:property name="base_height" value="0.05" />
+  <xacro:property name="base_height" value="0.12" />
   <xacro:property name="wheel_mass" value="0.3" /> <!-- arbitrary value for wheel mass -->
   <xacro:property name="wheel_len" value="0.040" />
@@ -49,5 +49,5 @@
       <parent link="${prefix}base_link"/>
       <child link="${prefix}left_wheel"/>
-      <origin xyz="${base_length/2} ${base_width/2} 0" rpy="${PI/2} 0 0"/>
+      <origin xyz="${base_length/2-wheel_radius} ${base_width/2 + (wheel_len/2) } 0" rpy="${PI/2} 0 0"/>
       <axis xyz="0 0 1"/>
       <dynamics damping="0.0"/>
@@ -78,5 +78,5 @@
       <parent link="${prefix}base_link"/>
       <child link="${prefix}right_wheel"/>
-      <origin xyz="${base_length/2} ${-base_width/2} 0" rpy="${PI/2} 0 0"/>
+      <origin xyz="${base_length/2-wheel_radius} ${-base_width/2  - (wheel_len/2) } 0" rpy="${PI/2} 0 0"/>
       <axis xyz="0 0 -1"/>
       <dynamics damping="0.0"/>
