Commit message: added gazebo ros2_control - with issues

File: description/urdf/diffbot.urdf.xacro (robot description, xacro)
@@ -9,7 +9,7 @@
   <xacro:include filename="$(find diffdrive_ddsm115)/urdf/diffbot.materials.xacro" />
   <!-- Import diffbot ros2_control description -->
-  <xacro:include filename="$(find diffdrive_ddsm115)/ros2_control/diffbot.ros2_control.xacro" />
+  <!-- <xacro:include filename="$(find diffdrive_ddsm115)/ros2_control/diffbot.ros2_control.xacro" /> -->
+  <xacro:include filename="$(find diffdrive_ddsm115)/ros2_control/gazebo.ros2_control.xacro" />
   <xacro:diffbot prefix="$(arg prefix)" />
-  <xacro:diffbot_ros2_control
-    name="DiffBot" prefix="$(arg prefix)" />
+  <xacro:diffbot_ros2_control name="DiffBot" prefix="$(arg prefix)" />
 </robot>

File: description/urdf/diffbot_description.urdf.xacro (robot description, xacro)
@@ -38,4 +38,7 @@
       </inertial>
     </link>
+    <gazebo reference="base_link">
+        <material>Gazebo/Green</material>
+    </gazebo>
     <!-- BASE_FOOTPRINT LINK -->
     <joint name="base_footprint_joint" type="fixed">
@@ -49,5 +52,5 @@
       <parent link="${prefix}base_link"/>
       <child link="${prefix}left_wheel"/>
-      <origin xyz="${base_length/2-wheel_radius} ${base_width/2 + (wheel_len/2) } 0" rpy="${PI/2} 0 0"/>
+      <origin xyz="${base_length/2-wheel_radius} ${base_width/2 + (wheel_len/2) } 0" rpy="-${PI/2} 0 0"/>
       <axis xyz="0 0 1"/>
       <dynamics damping="0.0"/>
@@ -75,4 +78,7 @@
       </inertial>
     </link>
+    <gazebo reference="left_wheel">
+        <material>Gazebo/Black</material>
+    </gazebo>
     <joint name="${prefix}right_wheel_joint" type="continuous">
       <parent link="${prefix}base_link"/>
@@ -102,6 +108,9 @@
           iyy="${wheel_mass / 12.0 * wheel_radius*wheel_radius}" iyz="0.0"
           izz="${wheel_mass / 12.0 * wheel_radius*wheel_radius}"/>
-        </inertial>
-      </link>
+      </inertial>
+    </link>
+    <gazebo reference="right_wheel">
+        <material>Gazebo/Black</material>
+    </gazebo>
     <joint name="${prefix}caster_rear_wheel_joint" type="fixed">
       <parent link="${prefix}base_link"/>

Commit message: Updated files for Ros2 control

File: description/urdf/diffbot.urdf.xacro (robot description, xacro)
@@ -2,6 +2,6 @@
 <!-- Basic differential drive mobile base -->
 <robot xmlns:xacro="http://www.ros.org/wiki/xacro" name="diffdrive_robot">
-  <!-- <xacro:include filename="robot_core.xacro" /> -->
-  <xacro:include filename="$(find diffdrive_ddsm115)/urdf/inertial_macros.xacro"/>
+  <xacro:arg name="prefix" default="" />
+  <!-- <xacro:include filename="$(find diffdrive_ddsm115)/urdf/inertial_macros.xacro"/> -->
   <xacro:include filename="$(find diffdrive_ddsm115)/urdf/diffbot_description.urdf.xacro" />
   <xacro:include filename="$(find diffdrive_ddsm115)/urdf/lidar.xacro" />
@@ -11,3 +11,6 @@
   <xacro:include filename="$(find diffdrive_ddsm115)/ros2_control/diffbot.ros2_control.xacro" />
   <!-- <xacro:include filename="$(find diffdrive_ddsm115)/ros2_control/gazebo.ros2_control.xacro" /> -->
+  <xacro:diffbot prefix="$(arg prefix)" />
+  <xacro:diffbot_ros2_control
+    name="DiffBot" prefix="$(arg prefix)" />
 </robot>

File: description/urdf/diffbot_description.urdf.xacro (robot description, xacro)
@@ -1,132 +1,161 @@
 <?xml version="1.0"?>
 <robot xmlns:xacro="http://www.ros.org/wiki/xacro">
+  <xacro:macro name="diffbot" params="prefix">
   <!-- Constants for robot dimensions -->
   <xacro:property name="PI" value="3.1415926535897931"/>
   <xacro:property name="base_mass" value="0.3" /> <!-- arbitrary value for base mass -->
-  <xacro:property name="base_width" value="0.15" />
-  <xacro:property name="base_length" value="0.3" />
-  <xacro:property name="base_height" value="0.12" />
+  <xacro:property name="base_width" value="0.1" />
+  <xacro:property name="base_length" value="0.1" />
+  <xacro:property name="base_height" value="0.05" />
   <xacro:property name="wheel_mass" value="0.3" /> <!-- arbitrary value for wheel mass -->
-  <xacro:property name="wheel_len" value="0.040" />
-  <xacro:property name="wheel_radius" value="0.05" />
+  <xacro:property name="wheel_len" value="0.020" />
+  <xacro:property name="wheel_radius" value="0.015" />
   <xacro:property name="caster_wheel_mass" value="0.1" /> <!-- arbitrary value for caster wheel mass -->
-  <xacro:property name="caster_wheel_radius" value="0.05" />
+  <xacro:property name="caster_wheel_radius" value="0.015" />
   <xacro:property name="z_offset" value="-${base_height/2}" /> <!-- Space btw top of beam and the each joint -->
   <!-- Base Link -->
-  <link name="base_link">
-  </link>
-  <!-- BASE_FOOTPRINT LINK -->
-  <joint name="base_footprint_joint" type="fixed">
-      <parent link="base_link"/>
-      <child link="base_footprint"/>
+  <link name="${prefix}base_link">
+    <collision>
       <origin xyz="0 0 0" rpy="0 0 0"/>
-  </joint>
-  <link name="base_footprint">
-  </link>
-  <!-- Chassis Link -->
-  <joint name="chassis_joint" type="fixed">
-    <parent link="base_link"/>
-    <child link="chassis"/>
-    <origin xyz="-0.1 0 0"/>
-  </joint>
-  <link name="chassis">
+      <geometry>
+        <box size="${base_width} ${base_length} ${base_height}"/>
+      </geometry>
+    </collision>
     <visual>
-        <origin xyz="${base_length/2} 0 ${base_height/2}"/>
+      <origin xyz="0 0 ${base_height/2}" rpy="0 0 0"/>
+      <geometry>
+        <box size="${base_width} ${base_length} ${base_height}"/>
+      </geometry>
+      <material name="orange"/>
+    </visual>
+    <inertial>
+      <origin xyz="0 0 0" rpy="0 0 0"/>
+      <mass value="${base_mass}"/>
+      <inertia
+        ixx="${base_mass / 12.0 * (base_length*base_length + base_height*base_height)}" ixy="0.0" ixz="0.0"
+        iyy="${base_mass / 12.0 * (base_height*base_height + base_width*base_width)}" iyz="0.0"
+        izz="${base_mass / 12.0 * (base_width*base_width + base_length*base_length)}"/>
+      </inertial>
+    </link>
+    <joint name="${prefix}left_wheel_joint" type="continuous">
+      <parent link="${prefix}base_link"/>
+      <child link="${prefix}left_wheel"/>
+      <origin xyz="0 -${base_width/2} ${z_offset}" rpy="0 0 0"/>
+      <axis xyz="0 1 0"/>
+      <dynamics damping="0.2"/>
+    </joint>
+    <!-- left wheel Link -->
+    <link name="${prefix}left_wheel">
+      <collision>
+        <origin xyz="0 0 0" rpy="${PI/2} 0 0"/>
         <geometry>
-            <box size="${base_length} ${base_width} ${base_height}"/>
+          <cylinder length="${wheel_len}" radius="${wheel_radius}"/>
+        </geometry>
+      </collision>
+      <visual>
+        <origin xyz="0 0 0" rpy="${PI/2} 0 0"/>
+        <geometry>
+          <cylinder length="${wheel_len}" radius="${wheel_radius}"/>
+        </geometry>
+        <material name="black"/>
+      </visual>
+      <inertial>
+        <origin xyz="0 0 0" rpy="${PI/2} 0 0"/>
+        <mass value="${wheel_mass}"/>
+        <inertia
+          ixx="${wheel_mass / 12.0 * (3*wheel_radius + wheel_len*wheel_len)}" ixy="0.0" ixz="0.0"
+          iyy="${wheel_mass / 12.0 * wheel_radius*wheel_radius}" iyz="0.0"
+          izz="${wheel_mass / 12.0 * wheel_radius*wheel_radius}"/>
+        </inertial>
+      </link>
+    <joint name="${prefix}right_wheel_joint" type="continuous">
+      <parent link="${prefix}base_link"/>
+      <child link="${prefix}right_wheel"/>
+      <origin xyz="0 ${base_width/2} ${z_offset}" rpy="0 0 0"/>
+      <axis xyz="0 1 0"/>
+      <dynamics damping="0.2"/>
+    </joint>
+    <!-- right wheel Link -->
+    <link name="${prefix}right_wheel">
+      <collision>
+        <origin xyz="0 0 0" rpy="${PI/2} 0 0"/>
+        <geometry>
+          <cylinder length="${wheel_len}" radius="${wheel_radius}"/>
+        </geometry>
+      </collision>
+      <visual>
+        <origin xyz="0 0 0" rpy="${PI/2} 0 0"/>
+        <geometry>
+          <cylinder length="${wheel_len}" radius="${wheel_radius}"/>
+        </geometry>
+        <material name="black"/>
+      </visual>
+      <inertial>
+        <origin xyz="0 0 0" rpy="${PI/2} 0 0"/>
+        <mass value="${wheel_mass}"/>
+        <inertia
+          ixx="${wheel_mass / 12.0 * (3*wheel_radius + wheel_len*wheel_len)}" ixy="0.0" ixz="0.0"
+          iyy="${wheel_mass / 12.0 * wheel_radius*wheel_radius}" iyz="0.0"
+          izz="${wheel_mass / 12.0 * wheel_radius*wheel_radius}"/>
+        </inertial>
+      </link>
+    <joint name="${prefix}caster_frontal_wheel_joint" type="fixed">
+      <parent link="${prefix}base_link"/>
+      <child link="${prefix}caster_frontal_wheel"/>
+      <origin xyz="${base_width/2 - caster_wheel_radius} 0 ${z_offset}" rpy="0 0 0"/>
+    </joint>
+    <!-- caster frontal wheel Link -->
+    <link name="${prefix}caster_frontal_wheel">
+      <collision>
+        <origin xyz="0 0 0" rpy="0 0 0"/>
+        <geometry>
+          <sphere radius="${caster_wheel_radius}"/>
+        </geometry>
+      </collision>
+      <visual>
+        <origin xyz="0 0 0" rpy="0 0 0"/>
+        <geometry>
+          <sphere radius="${caster_wheel_radius}"/>
         </geometry>
         <material name="white"/>
-    </visual>
-    <collision>
-          <origin xyz="${base_length/2} 0 ${base_height/2}"/>
+      </visual>
+      <inertial>
+        <origin xyz="0 0 0" rpy="0 0 0"/>
+        <mass value="${caster_wheel_mass}"/>
+        <inertia
+          ixx="${caster_wheel_mass * 0.4 * (caster_wheel_radius * caster_wheel_radius)}" ixy="0.0" ixz="0.0"
+          iyy="${caster_wheel_mass * 0.4 * (caster_wheel_radius * caster_wheel_radius)}" iyz="0.0"
+          izz="${caster_wheel_mass * 0.4 * (caster_wheel_radius * caster_wheel_radius)}"/>
+        </inertial>
+      </link>
+    <joint name="${prefix}caster_rear_wheel_joint" type="fixed">
+      <parent link="${prefix}base_link"/>
+      <child link="${prefix}caster_rear_wheel"/>
+      <origin xyz="${-base_width/2 + caster_wheel_radius} 0 ${z_offset}" rpy="0 0 0"/>
+    </joint>
+    <!-- caster rear wheel Link -->
+    <link name="${prefix}caster_rear_wheel">
+      <collision>
+        <origin xyz="0 0 0" rpy="0 0 0"/>
         <geometry>
-            <box size="${base_length} ${base_width} ${base_height}"/>
+          <sphere radius="${caster_wheel_radius}"/>
         </geometry>
-    </collision>
-    <xacro:inertial_box mass="${base_mass}" x="${base_length}" y="${base_width}" z="${base_height}">
-      <origin xyz="${base_length/2} 0 ${base_height/2}" rpy="0 0 0"/>
-    </xacro:inertial_box>
-  </link>
-  <gazebo reference="chassis">
-      <material>Gazebo/Green</material>
-  </gazebo>
-  <!-- left wheel Link -->
-  <joint name="left_wheel_joint" type="continuous">
-    <parent link="base_link"/>
-    <child link="left_wheel"/>
-    <origin xyz="0 ${base_width/2 + wheel_len/2} 0" rpy="-${PI/2} 0 0"/>
-    <axis xyz="0 0 1"/>
-  </joint>
-  <link name="left_wheel">
-    <visual>
-      <geometry>
-        <cylinder length="${wheel_len}" radius="${wheel_radius}"/>
-      </geometry>
-      <material name="black"/>
-    </visual>
-    <collision>
-      <geometry>
-        <cylinder length="${wheel_len}" radius="${wheel_radius}"/>
-      </geometry>
-    </collision>
-    <xacro:inertial_cylinder mass="${wheel_mass}" length="${wheel_len}" radius="${wheel_radius}">
-          <origin xyz="0 0 0" rpy="0 0 0"/>
-    </xacro:inertial_cylinder>
-  </link>
-  <gazebo reference="left_wheel">
-      <material>Gazebo/Black</material>
-  </gazebo>
-  <!-- right wheel Link -->
-  <joint name="right_wheel_joint" type="continuous">
-    <parent link="base_link"/>
-    <child link="right_wheel"/>
-    <origin xyz="0 -${base_width/2 + wheel_len/2} 0" rpy="${PI/2} 0 0"/>
-    <axis xyz="0 0 -1"/>
-  </joint>
-  <link name="right_wheel">
-    <visual>
-      <geometry>
-        <cylinder length="${wheel_len}" radius="${wheel_radius}"/>
-      </geometry>
-      <material name="black"/>
-    </visual>
-    <collision>
-      <geometry>
-        <cylinder length="${wheel_len}" radius="${wheel_radius}"/>
-      </geometry>
-    </collision>
-    <xacro:inertial_cylinder mass="${wheel_mass}" length="${wheel_len}" radius="${wheel_radius}">
-          <origin xyz="0 0 0" rpy="0 0 0"/>
-    </xacro:inertial_cylinder>
-  </link>
-  <gazebo reference="right_wheel">
-      <material>Gazebo/Black</material>
-  </gazebo>
-  <!-- caster rear wheel Link -->
-  <joint name="caster_rear_wheel_joint" type="fixed">
-    <parent link="chassis"/>
-    <child link="caster_rear_wheel"/>
-    <origin xyz="0.25 0 0"/>
-  </joint>
-  <link name="caster_rear_wheel">
-    <visual>
-      <geometry>
-        <sphere radius="${caster_wheel_radius}"/>
-      </geometry>
-      <material name="white"/>
-    </visual>
-    <collision>
-      <geometry>
-        <sphere radius="${caster_wheel_radius}"/>
-      </geometry>
-    </collision>
-    <xacro:inertial_sphere mass="0.1" radius="${caster_wheel_radius}">
-          <origin xyz="0 0 0" rpy="0 0 0"/>
-    </xacro:inertial_sphere>
-  </link>
-  <gazebo reference="caster_rear_wheel">
-    <material>Gazebo/White</material>
-    <mu1 value="0.001"/>
-    <mu2 value="0.001"/>
-  </gazebo>
+      </collision>
+      <visual>
+        <origin xyz="0 0 0" rpy="0 0 0"/>
+        <geometry>
+          <sphere radius="${caster_wheel_radius}"/>
+        </geometry>
+        <material name="white"/>
+      </visual>
+      <inertial>
+        <origin xyz="0 0 0" rpy="0 0 0"/>
+        <mass value="${caster_wheel_mass}"/>
+        <inertia
+          ixx="${caster_wheel_mass * 0.4 * (caster_wheel_radius * caster_wheel_radius)}" ixy="0.0" ixz="0.0"
+          iyy="${caster_wheel_mass * 0.4 * (caster_wheel_radius * caster_wheel_radius)}" iyz="0.0"
+          izz="${caster_wheel_mass * 0.4 * (caster_wheel_radius * caster_wheel_radius)}"/>
+        </inertial>
+      </link>
+  </xacro:macro>
 </robot>
