Commit message: Updated Lidar xacro

File: description/urdf/lidar.xacro (robot description, xacro)
@@ -4,5 +4,5 @@
         <parent link="base_link"/>
         <child link="laser_frame"/>
-        <origin xyz="0.1 0 0.125" rpy="0 0 0"/>
+        <origin xyz="0.1 0 0.125" rpy="0 0 3.1415926535897931"/>
     </joint>
     <link name="laser_frame">

Commit message: Updated lidar orientation in urdf

File: description/urdf/lidar.xacro (robot description, xacro)
@@ -4,5 +4,5 @@
         <parent link="chassis"/>
         <child link="laser_frame"/>
-        <origin xyz="0.122 0 0.212" rpy="0 0 0"/>
+        <origin xyz="0.122 0 0.212" rpy="0 0 -${PI/2}"/>
     </joint>
     <link name="laser_frame">

Commit message: Updated lidar urdf

File: description/urdf/lidar.xacro (robot description, xacro)
@@ -1,4 +1,5 @@
 <?xml version="1.0"?>
 <robot xmlns:xacro="http://www.ros.org/wiki/xacro" >
+    <xacro:property name="PI" value="3.1415926535897931"/>
     <joint name="laser_joint" type="fixed">
         <parent link="chassis"/>
