Commit message: Updated sim.launch and robot core

File: description/urdf/imu.xacro (robot description, xacro)
@@ -4,10 +4,10 @@
         <visual>
             <geometry>
-            <box size="0.1 0.1 0.1"/>
+            <box size="0.02 0.02 0.02"/>
             </geometry>
         </visual>
         <collision>
             <geometry>
-            <box size="0.1 0.1 0.1"/>
+            <box size="0.02 0.02 0.02"/>
             </geometry>
         </collision>
@@ -19,5 +19,5 @@
         <parent link="chassis"/>
         <child link="imu_link"/>
-        <origin xyz="0 0 0.01"/>
+        <origin xyz="0 0 0.1"/>
         </joint>
         <gazebo reference="imu_link">

File: description/urdf/robot_core.xacro (robot description, xacro)
@@ -5,10 +5,10 @@
     <xacro:property name="chassis_length" value="0.335"/>
     <xacro:property name="chassis_width" value="0.265"/>
-    <xacro:property name="chassis_height" value="0.138"/>
+    <xacro:property name="chassis_height" value="0.238"/>
     <xacro:property name="chassis_mass" value="1.0"/>
     <xacro:property name="wheel_radius" value="0.05125"/>
     <xacro:property name="wheel_thickness" value="0.04"/>
     <xacro:property name="wheel_mass" value="0.05"/>
-    <xacro:property name="wheel_offset_x" value="0.226"/>
+    <xacro:property name="wheel_offset_x" value="0.286"/>
     <xacro:property name="wheel_offset_y" value="0.115"/>
     <xacro:property name="wheel_offset_z" value="0.01"/>

Commit message: Update URDF

File: description/urdf/imu.xacro (robot description, xacro)
@@ -17,7 +17,7 @@
         </link>
         <joint name="imu_joint" type="fixed">
-        <parent link="chassis"/>
-        <child link="imu_link"/>
-        <origin xyz="0 0 0.1"/>
+            <parent link="base_link" />
+            <child link="imu_link" />
+            <origin xyz="0.08 0 0.17" />
         </joint>
         <gazebo reference="imu_link">

File: description/urdf/lidar.xacro (robot description, xacro)
@@ -3,7 +3,7 @@
     <xacro:property name="PI" value="3.1415926535897931"/>
     <joint name="laser_joint" type="fixed">
-        <parent link="chassis"/>
+        <parent link="base_link"/>
         <child link="laser_frame"/>
-        <origin xyz="0.042 0 0.212" rpy="0 0 -${PI/2}"/>
+        <origin xyz="-0.03 0 0.20" rpy="0 0 0"/>
     </joint>
     <link name="laser_frame">
@@ -12,12 +12,12 @@
                 <cylinder radius="0.05" length="0.04"/>
             </geometry>
-            <material name="black"/>
+            <material name="blue"/>
         </visual>
         <visual>
-            <origin xyz="0 0 -0.05"/>
+            <origin xyz="0 0 0.0"/>
             <geometry>
                 <cylinder radius="0.01" length="0.1"/>
             </geometry>
-            <material name="black"/>
+            <material name="blue"/>
         </visual>
         <collision>
@@ -31,5 +31,5 @@
     </link>
     <gazebo reference="laser_frame">
-        <material>Gazebo/Black</material>
+        <material>Gazebo/Blue</material>
         <sensor name="laser" type="ray">
             <pose> 0 0 0 0 0 0 </pose>

File: description/urdf/robot_core.xacro (robot description, xacro)
@@ -3,18 +3,18 @@
     <xacro:macro name="diffbot" params="prefix">
     <xacro:include filename="inertial_macros.xacro"/>
-    <xacro:property name="chassis_length" value="0.335"/>
-    <xacro:property name="chassis_width" value="0.265"/>
-    <xacro:property name="chassis_height" value="0.238"/>
+    <xacro:property name="chassis_length" value="0.27"/>
+    <xacro:property name="chassis_width" value="0.25"/>
+    <xacro:property name="chassis_height" value="0.09"/>
     <xacro:property name="chassis_mass" value="1.0"/>
-    <xacro:property name="wheel_radius" value="0.05125"/>
-    <xacro:property name="wheel_thickness" value="0.04"/>
+    <xacro:property name="wheel_radius" value="0.05035"/>
+    <xacro:property name="wheel_thickness" value="0.043"/>
     <xacro:property name="wheel_mass" value="0.05"/>
-    <xacro:property name="wheel_offset_x" value="0.286"/>
-    <xacro:property name="wheel_offset_y" value="0.115"/>
-    <xacro:property name="wheel_offset_z" value="0.01"/>
+    <xacro:property name="wheel_offset_x" value="-0.18"/>
+    <xacro:property name="wheel_offset_y" value="0.08"/>
+    <xacro:property name="wheel_offset_z" value="0.07"/>
     <xacro:property name="caster_wheel_radius" value="0.01"/>
     <xacro:property name="caster_wheel_mass" value="0.01"/>
-    <xacro:property name="caster_wheel_offset_x" value="0.075"/>
-    <xacro:property name="caster_wheel_offset_z" value="${wheel_offset_z - wheel_radius + caster_wheel_radius}"/>
+    <xacro:property name="caster_wheel_offset_x" value="0.055"/>
+    <xacro:property name="caster_wheel_offset_z" value="${-wheel_offset_z - wheel_radius + caster_wheel_radius}"/>
     <material name="white">
         <color rgba="1 1 1 1" />
@@ -47,5 +47,5 @@
         <parent link="base_link"/>
         <child link="chassis"/>
-        <origin xyz="${-wheel_offset_x} 0 ${-wheel_offset_z}"/>
+        <origin xyz="${wheel_offset_x} 0 ${wheel_offset_z}"/>
     </joint>
     <link name="chassis">
