Commit message: Updated diffdrive files

File: description/ros2_control/diffbot.ros2_control.xacro (robot description, xacro)
@@ -2,4 +2,5 @@
 <robot xmlns:xacro="http://www.ros.org/wiki/xacro">
   <xacro:macro name="diffbot_ros2_control" params="name prefix">
+  <xacro:unless value="$(arg sim_mode)">
     <ros2_control name="${name}" type="system">
       <hardware>
@@ -25,4 +26,34 @@
       </joint>
     </ros2_control>
+  </xacro:unless>
+  <xacro:if value="$(arg sim_mode)">
+    <ros2_control name="GazeboSystem" type="system">
+        <hardware>
+            <plugin>gazebo_ros2_control/GazeboSystem</plugin>
+        </hardware>
+        <joint name="${prefix}left_wheel_joint">
+            <command_interface name="velocity">
+                <param name="min">-10</param>
+                <param name="max">10</param>
+            </command_interface>
+            <state_interface name="velocity"/>
+            <state_interface name="position"/>
+        </joint>
+        <joint name="${prefix}right_wheel_joint">
+            <command_interface name="velocity">
+                <param name="min">-10</param>
+                <param name="max">10</param>
+            </command_interface>
+            <state_interface name="velocity"/>
+            <state_interface name="position"/>
+        </joint>
+    </ros2_control>
+    <gazebo>
+        <plugin name="gazebo_ros2_control" filename="libgazebo_ros2_control.so">
+            <parameters>$(find diffdrive_ddsm115)/config/diffbot_controllers.yaml</parameters>
+            <parameters>$(find diffdrive_ddsm115)/config/gaz_ros2_ctl_use_sim.yaml</parameters>
+        </plugin>
+    </gazebo>
+  </xacro:if>
   </xacro:macro>
 </robot>

File: description/urdf/diffbot.urdf.xacro (robot description, xacro)
@@ -3,12 +3,19 @@
 <robot xmlns:xacro="http://www.ros.org/wiki/xacro" name="diffdrive_robot">
   <xacro:arg name="prefix" default="" />
+  <xacro:arg name="use_ros2_control" default="true"/>
+  <xacro:arg name="sim_mode" default="false"/>
   <!-- <xacro:include filename="$(find diffdrive_ddsm115)/urdf/inertial_macros.xacro"/> -->
-  <xacro:include filename="$(find diffdrive_ddsm115)/urdf/diffbot_description.urdf.xacro" />
+  <!-- <xacro:include filename="$(find diffdrive_ddsm115)/urdf/diffbot_description.urdf.xacro" /> -->
+  <xacro:include filename="robot_core.xacro" />
   <!-- <xacro:include filename="$(find diffdrive_ddsm115)/urdf/lidar.xacro" /> -->
   <!-- Import Rviz colors -->
-  <xacro:include filename="$(find diffdrive_ddsm115)/urdf/diffbot.materials.xacro" />
+  <!-- <xacro:include filename="$(find diffdrive_ddsm115)/urdf/diffbot.materials.xacro" /> -->
   <!-- Import diffbot ros2_control description -->
-  <xacro:include filename="$(find diffdrive_ddsm115)/ros2_control/diffbot.ros2_control.xacro" />
-  <!-- <xacro:include filename="$(find diffdrive_ddsm115)/ros2_control/gazebo.ros2_control.xacro" /> -->
+  <xacro:if value="$(arg use_ros2_control)">
+    <xacro:include filename="$(find diffdrive_ddsm115)/ros2_control/diffbot.ros2_control.xacro" />
+  </xacro:if>
+  <xacro:unless value="$(arg use_ros2_control)">
+    <xacro:include filename="$(find diffdrive_ddsm115)/ros2_control/gazebo.ros2_control.xacro" />
+  </xacro:unless>
   <xacro:diffbot prefix="$(arg prefix)" />
   <xacro:diffbot_ros2_control

File: description/urdf/diffbot_description.urdf.xacro (robot description, xacro)
@@ -4,14 +4,14 @@
   <!-- Constants for robot dimensions -->
   <xacro:property name="PI" value="3.1415926535897931"/>
-  <xacro:property name="base_mass" value="0.3" /> <!-- arbitrary value for base mass -->
-  <xacro:property name="base_width" value="0.1" />
-  <xacro:property name="base_length" value="0.1" />
-  <xacro:property name="base_height" value="0.05" />
-  <xacro:property name="wheel_mass" value="0.3" /> <!-- arbitrary value for wheel mass -->
-  <xacro:property name="wheel_len" value="0.020" />
-  <xacro:property name="wheel_radius" value="0.015" />
+  <xacro:property name="base_mass" value="1.0" /> <!-- arbitrary value for base mass -->
+  <xacro:property name="base_width" value="0.265" />
+  <xacro:property name="base_length" value="0.335" />
+  <xacro:property name="base_height" value="0.138" />
+  <xacro:property name="wheel_mass" value="0.05" /> <!-- arbitrary value for wheel mass -->
+  <xacro:property name="wheel_len" value="0.026" />
+  <xacro:property name="wheel_radius" value="0.033" />
   <xacro:property name="caster_wheel_mass" value="0.1" /> <!-- arbitrary value for caster wheel mass -->
   <xacro:property name="caster_wheel_radius" value="0.015" />
-  <xacro:property name="z_offset" value="-${base_height/2}" /> <!-- Space btw top of beam and the each joint -->
+  <xacro:property name="z_offset" value="-${base_height/2 - (caster_wheel_radius*2) }" /> <!-- Space btw top of beam and the each joint -->
   <!-- Base Link -->
   <link name="${prefix}base_link">
@@ -129,4 +129,9 @@
         </inertial>
       </link>
+      <gazebo reference="${prefix}caster_frontal_wheel">
+        <material>Gazebo/White</material>
+        <mu1 value="0.001"/>
+        <mu2 value="0.001"/>
+      </gazebo>
     <joint name="${prefix}caster_rear_wheel_joint" type="fixed">
       <parent link="${prefix}base_link"/>
@@ -158,4 +163,9 @@
         </inertial>
       </link>
+      <gazebo reference="${prefix}caster_rear_wheel">
+        <material>Gazebo/White</material>
+        <mu1 value="0.001"/>
+        <mu2 value="0.001"/>
+      </gazebo>
   </xacro:macro>
 </robot>

File: description/urdf/robot_core.xacro (robot description, xacro)
@@ -1,5 +1,20 @@
 <?xml version="1.0"?>
 <robot xmlns:xacro="http://www.ros.org/wiki/xacro" >
+    <xacro:macro name="diffbot" params="prefix">
     <xacro:include filename="inertial_macros.xacro"/>
+    <xacro:property name="chassis_length" value="0.335"/>
+    <xacro:property name="chassis_width" value="0.265"/>
+    <xacro:property name="chassis_height" value="0.138"/>
+    <xacro:property name="chassis_mass" value="1.0"/>
+    <xacro:property name="wheel_radius" value="0.033"/>
+    <xacro:property name="wheel_thickness" value="0.026"/>
+    <xacro:property name="wheel_mass" value="0.05"/>
+    <xacro:property name="wheel_offset_x" value="0.226"/>
+    <xacro:property name="wheel_offset_y" value="0.1485"/>
+    <xacro:property name="wheel_offset_z" value="0.01"/>
+    <xacro:property name="caster_wheel_radius" value="0.01"/>
+    <xacro:property name="caster_wheel_mass" value="0.01"/>
+    <xacro:property name="caster_wheel_offset_x" value="0.075"/>
+    <xacro:property name="caster_wheel_offset_z" value="${wheel_offset_z - wheel_radius + caster_wheel_radius}"/>
     <material name="white">
         <color rgba="1 1 1 1" />
@@ -15,5 +30,5 @@
     </material>
     <material name="red">
-        <color rgba="1 0 0 "/>
+        <color rgba="1 0 0 1"/>
     </material>
     <!-- BASE LINK -->
@@ -32,26 +47,26 @@
         <parent link="base_link"/>
         <child link="chassis"/>
-        <origin xyz="-0.1 0 0"/>
+        <origin xyz="${-wheel_offset_x} 0 ${-wheel_offset_z}"/>
     </joint>
     <link name="chassis">
         <visual>
-            <origin xyz="0.15 0 0.075"/>
+            <origin xyz="${chassis_length/2} 0 ${chassis_height/2}"/>
             <geometry>
-                <box size="0.3 0.3 0.15"/>
+                <box size="${chassis_length} ${chassis_width} ${chassis_height}"/>
             </geometry>
-            <material name="white"/>
+            <material name="orange"/>
         </visual>
         <collision>
-            <origin xyz="0.15 0 0.075"/>
+            <origin xyz="${chassis_length/2} 0 ${chassis_height/2}"/>
             <geometry>
-                <box size="0.3 0.3 0.15"/>
+                <box size="${chassis_length} ${chassis_width} ${chassis_height}"/>
             </geometry>
         </collision>
-        <xacro:inertial_box mass="0.5" x="0.3" y="0.3" z="0.15">
-            <origin xyz="0.15 0 0.075" rpy="0 0 0"/>
+        <xacro:inertial_box mass="0.5" x="${chassis_length}" y="${chassis_width}" z="${chassis_height}">
+            <origin xyz="${chassis_length/2} 0 ${chassis_height/2}" rpy="0 0 0"/>
         </xacro:inertial_box>
     </link>
     <gazebo reference="chassis">
-        <material>Gazebo/White</material>
+        <material>Gazebo/Orange</material>
     </gazebo>
     <!-- LEFT WHEEL LINK -->
@@ -59,5 +74,5 @@
         <parent link="base_link"/>
         <child link="left_wheel"/>
-        <origin xyz="0 0.175 0" rpy="-${pi/2} 0 0" />
+        <origin xyz="0 ${wheel_offset_y} 0" rpy="-${pi/2} 0 0" />
         <axis xyz="0 0 1"/>
     </joint>
@@ -65,5 +80,5 @@
         <visual>
             <geometry>
-                <cylinder radius="0.05" length="0.04"/>
+                <cylinder radius="${wheel_radius}" length="${wheel_thickness}"/>
             </geometry>
             <material name="blue"/>
@@ -71,8 +86,8 @@
         <collision>
             <geometry>
-                <cylinder radius="0.05" length="0.04"/>
+                <sphere radius="${wheel_radius}"/>
             </geometry>
         </collision>
-        <xacro:inertial_cylinder mass="0.1" length="0.04" radius="0.05">
+        <xacro:inertial_cylinder mass="${wheel_mass}" length="${wheel_thickness}" radius="${wheel_radius}">
             <origin xyz="0 0 0" rpy="0 0 0"/>
         </xacro:inertial_cylinder>
@@ -85,5 +100,5 @@
         <parent link="base_link"/>
         <child link="right_wheel"/>
-        <origin xyz="0 -0.175 0" rpy="${pi/2} 0 0" />
+        <origin xyz="0 ${-wheel_offset_y} 0" rpy="${pi/2} 0 0" />
         <axis xyz="0 0 -1"/>
     </joint>
@@ -91,5 +106,5 @@
         <visual>
             <geometry>
-                <cylinder radius="0.05" length="0.04"/>
+                <cylinder radius="${wheel_radius}" length="${wheel_thickness}"/>
             </geometry>
             <material name="blue"/>
@@ -97,8 +112,8 @@
         <collision>
             <geometry>
-                <cylinder radius="0.05" length="0.04"/>
+                <sphere radius="${wheel_radius}"/>
             </geometry>
         </collision>
-        <xacro:inertial_cylinder mass="0.1" length="0.04" radius="0.05">
+        <xacro:inertial_cylinder mass="${wheel_mass}" length="${wheel_thickness}" radius="${wheel_radius}">
             <origin xyz="0 0 0" rpy="0 0 0"/>
         </xacro:inertial_cylinder>
@@ -111,26 +126,27 @@
         <parent link="chassis"/>
         <child link="caster_wheel"/>
-        <origin xyz="0.24 0 0"/>
+        <origin xyz="${caster_wheel_offset_x} 0 ${caster_wheel_offset_z}"/>
     </joint>
     <link name="caster_wheel">
         <visual>
             <geometry>
-                <sphere radius="0.05"/>
+                <sphere radius="${caster_wheel_radius}"/>
             </geometry>
-            <material name="black"/>
+            <material name="white"/>
         </visual>
         <collision>
             <geometry>
-                <sphere radius="0.05"/>
+                <sphere radius="${caster_wheel_radius}"/>
             </geometry>
         </collision>
-        <xacro:inertial_sphere mass="0.1" radius="0.05">
+        <xacro:inertial_sphere mass="${caster_wheel_mass}" radius="${caster_wheel_radius}">
             <origin xyz="0 0 0" rpy="0 0 0"/>
         </xacro:inertial_sphere>
     </link>
     <gazebo reference="caster_wheel">
-        <material>Gazebo/Black</material>
+        <material>Gazebo/White</material>
         <mu1 value="0.001"/>
         <mu2 value="0.001"/>
     </gazebo>
+    </xacro:macro>
 </robot>

Commit message: Updated some params for nav2

File: description/ros2_control/diffbot.ros2_control.xacro (robot description, xacro)
@@ -8,5 +8,5 @@
         <param name="left_wheel_name">left_wheel_joint</param>
         <param name="right_wheel_name">right_wheel_joint</param>
-        <param name="device">/dev/serial/by-id/usb-FTDI_FT232R_USB_UART_AQ0288O8-if00-port0</param>
+        <param name="ddsm115_device">/dev/serial/by-id/usb-FTDI_FT232R_USB_UART_AQ0288O8-if00-port0</param>
         <!-- <param name="device">/dev/ttyUSB1</param> -->
         <param name="baud_rate">115200</param>

File: description/urdf/diffbot.urdf.xacro (robot description, xacro)
@@ -5,8 +5,8 @@
   <xacro:arg name="use_ros2_control" default="true"/>
   <xacro:arg name="sim_mode" default="false"/>
-  <!-- <xacro:include filename="$(find diffdrive_ddsm115)/urdf/inertial_macros.xacro"/> -->
+  <xacro:include filename="$(find diffdrive_ddsm115)/urdf/inertial_macros.xacro"/>
   <!-- <xacro:include filename="$(find diffdrive_ddsm115)/urdf/diffbot_description.urdf.xacro" /> -->
   <xacro:include filename="robot_core.xacro" />
-  <!-- <xacro:include filename="$(find diffdrive_ddsm115)/urdf/lidar.xacro" /> -->
+  <xacro:include filename="$(find diffdrive_ddsm115)/urdf/lidar.xacro" />
   <!-- Import Rviz colors -->
   <!-- <xacro:include filename="$(find diffdrive_ddsm115)/urdf/diffbot.materials.xacro" /> -->

File: description/urdf/lidar.xacro (robot description, xacro)
@@ -2,14 +2,21 @@
 <robot xmlns:xacro="http://www.ros.org/wiki/xacro" >
     <joint name="laser_joint" type="fixed">
-        <parent link="base_link"/>
+        <parent link="chassis"/>
         <child link="laser_frame"/>
-        <origin xyz="0.1 0 0.125" rpy="0 0 3.1415926535897931"/>
+        <origin xyz="0.122 0 0.212" rpy="0 0 0"/>
     </joint>
     <link name="laser_frame">
         <visual>
             <geometry>
-                <cylinder radius="0.03" length="0.04"/>
+                <cylinder radius="0.05" length="0.04"/>
             </geometry>
-            <material name="red"/>
+            <material name="black"/>
+        </visual>
+        <visual>
+            <origin xyz="0 0 -0.05"/>
+            <geometry>
+                <cylinder radius="0.01" length="0.1"/>
+            </geometry>
+            <material name="black"/>
         </visual>
         <collision>
@@ -23,5 +30,5 @@
     </link>
     <gazebo reference="laser_frame">
-        <material>Gazebo/Red</material>
+        <material>Gazebo/Black</material>
         <sensor name="laser" type="ray">
             <pose> 0 0 0 0 0 0 </pose>

Commit message: Added robot_localization

File: description/ros2_control/diffbot.ros2_control.xacro (robot description, xacro)
@@ -17,4 +17,6 @@
         <param name="imu_device">/dev/serial/by-id/usb-Arduino_Seeed_XIAO_nRF52840_Sense_D1CD2B3275EB486A-if00</param>
         <param name="imu_baud_rate">57600</param>
+        <param name='sensor_name'>imu_sensor</param>
+        <param name='frame_id'>imu_link</param>
       </hardware>
       <!-- Wheel Interfaces -->
@@ -30,5 +32,5 @@
       </joint>
       <!-- IMU Interfaces -->
-      <sensor name="${prefix}imu_joint">
+      <sensor name="imu_sensor">
         <!-- Quaternion Interfaces -->
         <state_interface name="orientation.x"/>
@@ -44,5 +46,4 @@
         <state_interface name="linear_acceleration.y"/>
         <state_interface name="linear_acceleration.z"/>
-        <param name="frame_id">imu_link</param>
       </sensor>
     </ros2_control>

File: description/urdf/lidar.xacro (robot description, xacro)
@@ -5,5 +5,5 @@
         <parent link="chassis"/>
         <child link="laser_frame"/>
-        <origin xyz="0.122 0 0.212" rpy="0 0 -${PI/2}"/>
+        <origin xyz="0.042 0 0.212" rpy="0 0 -${PI/2}"/>
     </joint>
     <link name="laser_frame">
